File: ch32v003-512.kicad_sch (KiCad schematic)
At the start: 0 parts

Commit message: upload 2
Other:
- sheet col_0 ports: added COL0_PWR_GOOD; removed 3V3_COL
- sheet col_1 ports: added COL1_PWR_GOOD; removed 3V3_COL
- sheet col_2 ports: added COL2_PWR_GOOD; removed 3V3_COL
- sheet col_3 ports: added COL3_PWR_GOOD; removed 3V3_COL
- sheet host_mcu ports: added SPI_CS_COL1; removed SPI_CS_COl1
Changed lines of the file:
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@@
 			)
 		)
-		(pin "3V3_COL" output
+		(pin "COL2_PWR_GOOD" output
 			(at 511.81 59.69 90)
 			(effects
@@
 			)
 		)
-		(pin "3V3_COL" output
+		(pin "COL1_PWR_GOOD" output
 			(at 353.06 59.69 90)
 			(effects
@@
 			)
 		)
-		(pin "SPI_CS_COl1" output
+		(pin "SPI_CS_COL1" output
 			(at 130.81 388.62 0)
 			(effects
@@
 			)
 		)
-		(pin "3V3_COL" output
+		(pin "COL3_PWR_GOOD" output
 			(at 665.48 59.69 90)
 			(effects
@@
 			)
 		)
-		(pin "3V3_COL" output
+		(pin "COL0_PWR_GOOD" output
 			(at 199.39 59.69 90)
 			(effects

Commit message: upload 3
Other:
- sheet backplane_power ports: added 3V3_MAIN, 5V_ATX; removed 3V3, 5V
- sheet col_0 ports: added none; removed COL0_PWR_GOOD
- sheet col_1 ports: added none; removed COL1_PWR_GOOD
- sheet col_2 ports: added none; removed COL2_PWR_GOOD
- sheet col_3 ports: added none; removed COL3_PWR_GOOD
Changed lines of the file:
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@@
-			)
-		)
-		(pin "COL2_PWR_GOOD" output
-			(at 511.81 59.69 90)
-			(effects
-				(font
-					(size 1.27 1.27)
-				)
-				(justify right)
 			)
 		)
@@
 			)
 		)
-		(pin "COL1_PWR_GOOD" output
-			(at 353.06 59.69 90)
-			(effects
-				(font
-					(size 1.27 1.27)
-				)
-				(justify right)
-			)
-		)
 		(pin "5V_ATX" input
 			(at 355.6 59.69 90)
@@
 			)
 		)
-		(pin "3V3" output
+		(pin "3V3_MAIN" output
 			(at 351.79 466.09 0)
 			(effects
@@
 			)
 		)
-		(pin "5V" output
+		(pin "5V_ATX" output
 			(at 351.79 468.63 0)
 			(effects
@@
 			)
 		)
-		(pin "COL3_PWR_GOOD" output
-			(at 665.48 59.69 90)
-			(effects
-				(font
-					(size 1.27 1.27)
-				)
-				(justify right)
-			)
-		)
 		(pin "5V_ATX" input
 			(at 668.02 59.69 90)
@@
 			)
 		)
-		(pin "COL0_PWR_GOOD" output
-			(at 199.39 59.69 90)
-			(effects
-				(font
-					(size 1.27 1.27)
-				)
-				(justify right)
-			)
-		)

Commit message: upload 4
Parts:
- added J4, J5, J8, J9: Bus_M.2_Socket_B, symbol Connector:Bus_M.2_Socket_B
Connections:
- net 3V3_MAIN: now also J4.2 (3.3V), J4.4 (3.3V), J4.70 (3.3V), J4.72 (3.3V), J4.74 (3.3V), J5.2 (3.3V), J5.4 (3.3V), J5.70 (3.3V), J5.72 (3.3V), J5.74 (3.3V), J8.2 (3.3V), J8.4 (3.3V), J8.70 (3.3V), J8.72 (3.3V), J8.74 (3.3V), J9.2 (3.3V), J9.4 (3.3V), J9.70 (3.3V), J9.72 (3.3V), J9.74 (3.3V)
- net PWR_GOOD: now also J4.6 (~{FULL_CARD_POWER_OFF}), J5.6 (~{FULL_CARD_POWER_OFF}), J8.6 (~{FULL_CARD_POWER_OFF}), J9.6 (~{FULL_CARD_POWER_OFF})
- net SPI_CS_COL0: now also J8.46 (GPIO_3)
- net SPI_CS_COL1: now also J4.46 (GPIO_3)
- net SPI_CS_COL2: now also J5.46 (GPIO_3)
- net SPI_CS_COL3: now also J9.46 (GPIO_3)
- net SPI_H_CLK: now also J4.40 (GPIO_0), J5.40 (GPIO_0), J8.40 (GPIO_0), J9.40 (GPIO_0)
- net SPI_H_MISO: now also J4.44 (GPIO_2), J5.44 (GPIO_2), J8.44 (GPIO_2), J9.44 (GPIO_2)
- net SPI_H_MOSI: now also J4.42 (GPIO_1), J5.42 (GPIO_1), J8.42 (GPIO_1), J9.42 (GPIO_1)
- net SYS_FAULT: now also J4.48 (GPIO_4), J5.48 (GPIO_4), J8.48 (GPIO_4), J9.48 (GPIO_4)
- net SYS_NRST: now also J4.20 (GPIO_5), J4.50 (~{PERST}), J4.67 (~{RESET}), J5.20 (GPIO_5), J5.50 (~{PERST}), J5.67 (~{RESET}), J8.20 (GPIO_5), J8.50 (~{PERST}), J8.67 (~{RESET}), J9.20 (GPIO_5), J9.50 (~{PERST}), J9.67 (~{RESET})
- net backplane_power/GND: now also J4.11 (GND), J4.27 (GND), J4.3 (GND), J4.33 (GND), J4.39 (GND), J4.45 (GND), J4.5 (GND), J4.51 (GND), J4.57 (GND), J4.71 (GND), J4.73 (GND), J5.11 (GND), J5.27 (GND), J5.3 (GND), J5.33 (GND), J5.39 (GND), J5.45 (GND), J5.5 (GND), J5.51 (GND), J5.57 (GND), J5.71 (GND), J5.73 (GND), J8.11 (GND), J8.27 (GND), J8.3 (GND), J8.33 (GND), J8.39 (GND), J8.45 (GND), J8.5 (GND), J8.51 (GND), J8.57 (GND), J8.71 (GND), J8.73 (GND), J9.11 (GND), J9.27 (GND), J9.3 (GND), J9.33 (GND), J9.39 (GND), J9.45 (GND), J9.5 (GND), J9.51 (GND), J9.57 (GND), J9.71 (GND), J9.73 (GND)
- no-connect marks 0 -> 160
Other:
- removed sheet col_0
- removed sheet col_1
- removed sheet col_2
- removed sheet col_3
- sheet host_mcu ports: added none; removed USB_DM, USB_DP
- note added: "J-COL0"
- note added: "J-COL1"
- note added: "J-COL2"
- note added: "J-COL3"
