File: column.kicad_sch (KiCad schematic)
At the start: 0 parts

Commit message: upload 2
Changed lines of the file:
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@@
 		)
 	)
-	(hierarchical_label "3V3_COL"
+	(hierarchical_label "COL_PWR_GOOD"
 		(shape output)
 		(at 273.05 31.75 0)

Commit message: upload 3
Changed lines of the file:
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@@
-		)
-	)
-	(hierarchical_label "COL_PWR_GOOD"
-		(shape output)
-		(at 273.05 31.75 0)
-		(effects
-			(font
-				(size 1.27 1.27)
-			)
-			(justify left)
 		)
 	)

Commit message: upload 4
Parts:
- added J4: Bus_M.2_Socket_E, symbol Connector:Bus_M.2_Socket_E
Connections:
- net SPI_H_CLK: now also J4.9 (SDIO_CLK)
- new net: J4.1 (GND), J4.18 (GND), J4.33 (GND), J4.39 (GND), J4.45 (GND), J4.51 (GND), J4.57 (GND), J4.63 (GND), J4.69 (GND), J4.7 (GND), J4.75 (GND)
- new net: J4.2 (3.3V), J4.4 (3.3V), J4.72 (3.3V), J4.74 (3.3V)
Changed lines of the file:
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@@
 	(hierarchical_label "SYS_NRST"
 		(shape input)
-		(at 273.05 24.13 0)
+		(at 95.25 46.99 0)
 		(effects
 			(font
@@
 	(hierarchical_label "5V_ATX"
 		(shape input)
-		(at 273.05 29.21 0)
+		(at 95.25 52.07 0)
 		(effects
 			(font
@@
 	(hierarchical_label "SPI_CS"
 		(shape input)
-		(at 273.05 21.59 0)
+		(at 95.25 44.45 0)
 		(effects
 			(font
@@
 	(hierarchical_label "SPI_H_MISO"
 		(shape output)
-		(at 273.05 19.05 0)
+		(at 95.25 41.91 0)
 		(effects
 			(font
@@
 	(hierarchical_label "SPI_H_CLK"
 		(shape input)
-		(at 273.05 13.97 0)
-		(effects
-			(font
-				(size 1.27 1.27)
-			)
-			(justify left)
+		(at 143.51 88.9 180)
+		(effects
+			(font
+				(size 1.27 1.27)
+			)
+			(justify right)
 		)
 	)
 	(hierarchical_label "SYS_FAULT"
 		(shape bidirectional)
-		(at 273.05 26.67 0)
+		(at 95.25 49.53 0)
 		(effects
 			(font
@@
 	(hierarchical_label "SPI_H_MOSI"
 		(shape input)
-		(at 273.05 16.51 0)
-		(effects
-			(font
-				(size 1.27 1.27)
-			)
-			(justify left)
-		)
-	)
+		(at 95.25 39.37 0)
+		(effects
+			(font
+				(size 1.27 1.27)
+			)
+			(justify left)
+		)
+	)
+	(symbol
+		(lib_id "Connector:Bus_M.2_Socket_E")
+		(at 168.91 76.2 0)
+		(unit 1)
+		(exclude_from_sim no)
+		(in_bom yes)
+		(on_board yes)
+		(dnp no)
+		(property "Reference" "J4"
+			(at 171.0533 25.4 0)
+			(effects
+				(font
+					(size 1.27 1.27)
+				)
+				(justify left)
+			)
+		)
+		(property "Value" "Bus_M.2_Socket_E"
+			(at 171.0533 27.94 0)
+			(effects
+				(font
+					(size 1.27 1.27)
+				)
+				(justify left)
+			)
+		)
+		(property "Footprint" ""
+			(at 168.91 49.53 0)
+			(effects
+				(font
+					(size 1.27 1.27)
+				)
+				(hide yes)
+			)
+		)
+		(property "Datasheet" "https://web.archive.org/web/20200613074028/http://read.pudn.com/downloads794/doc/project/3133918/PCIe_M.2_Electromechanical_Spec_Rev1.0_Final_11012013_RS_Clean.pdf#page=150"
+			(at 168.91 63.5 0)
+			(effects
+				(font
+					(size 1.27 1.27)
+				)
+				(hide yes)
+			)
+		)
+		(property "Description" "M.2 Socket 1-SD Mechanical Key E"
+			(at 168.91 76.2 0)
+			(effects
+				(font
+					(size 1.27 1.27)
+				)
+				(hide yes)
+			)
+		)
+		(pin "62"
+		)
+		(pin "53"
+		)
+		(pin "37"
+		)
+		(pin "43"
+		)
+		(pin "70"
+		)
+		(pin "72"
+		)
+		(pin "45"
+		)
+		(pin "69"
+		)
+		(pin "52"
+		)
+		(pin "61"
+		)
+		(pin "13"
+		)
+		(pin "17"
+		)
+		(pin "7"
+		)
+		(pin "58"
+		)
+		(pin "51"
+		)
+		(pin "57"
+		)
+		(pin "71"
+		)
+		(pin "35"
+		)
+		(pin "75"
+		)
+		(pin "60"
+		)
+		(pin "9"
+		)
+		(pin "4"
+		)
+		(pin "1"
+		)
+		(pin "55"
+		)
+		(pin "41"
+		)
+		(pin "65"
+		)
+		(pin "68"
+		)
+		(pin "15"
+		)
+		(pin "73"
+		)
+		(pin "2"
+		)
+		(pin "67"
+		)
+		(pin "5"
+		)
+		(pin "11"
+		)
+		(pin "19"
+		)
+		(pin "66"
+		)
+		(pin "21"
+		)
+		(pin "3"
+		)
+		(pin "59"
+		)
+		(pin "49"
+		)
+		(pin "18"
+		)
+		(pin "33"
+		)
+		(pin "39"
+		)
+		(pin "63"
+		)
+		(pin "47"
+		)
+		(pin "64"
+		)
+		(pin "38"
+		)
+		(pin "23"
+		)
+		(pin "74"
+		)
+		(pin "40"
+		)
+		(pin "42"
+		)
+		(pin "54"
+		)
+		(pin "8"
+		)
+		(pin "10"
+		)
+		(pin "12"
+		)
+		(pin "14"
+		)
+		(pin "22"
+		)
+		(pin "32"
+		)
+		(pin "20"
+		)
+		(pin "34"
+		)
+		(pin "56"
+		)
+		(pin "36"
+		)
+		(pin "6"
+		)
+		(pin "50"
+		)
+		(pin "46"
+		)
+		(pin "44"
+		)
+		(pin "16"
+		)
+		(pin "48"
+		)
+		(instances
+			(project ""
+				(path "/5e6c9623-e737-45ef-bb1f-893413b06cbf/0276f070-05cd-4ac9-a010-ce24c4c80ca1"
+					(reference "J6")
+					(unit 1)
+				)
+				(path "/5e6c9623-e737-45ef-bb1f-893413b06cbf/7a544113-dc97-4dca-96e8-b3ec478d9f40"
+					(reference "J4")
+					(unit 1)
+				)
+				(path "/5e6c9623-e737-45ef-bb1f-893413b06cbf/c41a39bb-4d27-400b-9ac0-37562a1db907"
+					(reference "J7")
+					(unit 1)
+				)
+				(path "/5e6c9623-e737-45ef-bb1f-893413b06cbf/c4cdeaa7-02f2-48f5-8115-a522dd175833"
+					(reference "J5")
+					(unit 1)
+				)
+			)
+		)
+	)
