File: host.kicad_sch (KiCad schematic)
At the start: 0 parts

Commit message: upload 2
Changed lines of the file:
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@@
 		)
 	)
-	(hierarchical_label "SPI_CS_COl1"
+	(hierarchical_label "SPI_CS_COL1"
 		(shape output)
 		(at 267.97 82.55 0)

Commit message: upload 3
Parts:
- added C10, C4, C6, C7, C8: 100nF, symbol Device:C
- added C11, C12: 20pF, symbol Device:C
- added C5: 4.7uF, symbol Device:C
- added C9: 1uF, symbol Device:C
- added J2: USB_C_Receptacle_USB2.0_14P, symbol Connector:USB_C_Receptacle_USB2.0_14P
- added R4, R5: 10k, symbol Device:R
- added R6: 1M, symbol Device:R
- added R7, R8: 5.1k, symbol Device:R
- added R9: 100k, symbol Device:R
- added U2: CH32V30xRxTx, Package_QFP:LQFP-64_10x10mm_P0.5mm, symbol MCU_WCH_RiscV:CH32V30xRxTx
- added U3: USBLC6-2SC6, Package_TO_SOT_SMD:SOT-23-6, symbol Power_Protection:USBLC6-2SC6
- added Y1: 8MHz, symbol Device:Crystal
Connections:
- new net: C11.2, Y1.1
- new net: C12.2, Y1.2
- new net: C12.1, R6.2, U2.6 (OSC_OUT)
- new net: C11.1, R6.1, U2.5 (OSC_IN)
- new net: R5.1, U2.60 (BOOT0)
- new net: C10.2, R4.2, U2.7 (~{RST})
- new net: J2.A5 (CC1), R7.1
- new net: J2.B5 (CC2), R8.1
- new net +3V3: C4.1, C5.1, C6.1, C7.2, C8.1, C9.1, R4.1, U2.1 (VBAT), U2.13 (VDDA), U2.19 (VDD), U2.32 (VIO), U2.48 (VDD), U2.64 (VIO)
- new net +5V: J2.A4 (VBUS), J2.A9 (VBUS), J2.B4 (VBUS), J2.B9 (VBUS), R9.2, U3.4 (I/O2)
- new net GND: C10.1, C4.2, C5.2, C6.2, C7.1, C8.2, C9.2, J2.A1 (GND), J2.A12 (GND), J2.B1 (GND), J2.B12 (GND), J2.S1 (SHIELD), R5.2, R7.2, R8.2, R9.1, U2.12 (VSSA), U2.18 (VSS), U2.31 (VSS), U2.47 (VSS), U2.63 (VSS), U3.2 (GND)
- no-connect marks 0 -> 2

Commit message: upload 3
Parts:
- added J3: DEBUG, symbol Connector_Generic:Conn_01x05
- added R10, R11: 22o, symbol Device:R
Connections:
- net +3V3: now also J3.1 (Pin_1)
- net GND: now also J3.5 (Pin_5)
- net SPI_CS_COL0: now also U2.20 (PA4)
- net SPI_CS_COL1: now also U2.17 (PA3)
- net SPI_CS_COL2: now also U2.16 (PA2)
- net SPI_CS_COL3: now also U2.15 (PA1)
- net SPI_H_CLK: now also U2.21 (PA5)
- net SPI_H_MISO: now also U2.22 (PA6)
- net SPI_H_MOSI: now also U2.23 (PA7)
- net SYS_FAULT: now also U2.9 (PC1)
- net SYS_NRST: now also U2.8 (PC0)
- net at U2.44 (PA11): now also U3.1 (I/O1), U3.6 (I/O1), R11.2
- net at U2.45 (PA12): now also U3.3 (I/O2), U3.5 (VBUS), R10.2
- net at U2.46 (SWDIO): now also J3.2 (Pin_2)
- net at U2.49 (SWCLK): now also J3.3 (Pin_3)
- net NRST_HOST: now reaches C10.2, R4.2, U2.7 (~{RST})
- net NRST_HOST: now also J3.4 (Pin_4)
- net at J2.A6 (D+): now also J2.B6 (D+), R10.1
- net at J2.A7 (D-): now also J2.B7 (D-), R11.1
- no-connect marks 2 -> 36

Commit message: upload 4
Connections:
- net +5V: no longer J2.A4 (VBUS), J2.A9 (VBUS), J2.B4 (VBUS), J2.B9 (VBUS), R9.2
- net +3V3 renamed 3V3_MAIN
- new net: J2.A4 (VBUS), J2.A9 (VBUS), J2.B4 (VBUS), J2.B9 (VBUS), R9.2
